File: protoA/protoA.kicad_sch (KiCad schematic)
At the start: 30 parts, among them U1 W65C816SxP, U10 74LS02, U2 RaspberryPi_Pico, U3 ESP-PSRAM64H, U4 ESP-PSRAM64H, U5 SN74LVC245APW, U6 SN74LVC245APW, U7 SN74LVC245APW, U8 74HC139, U9 74AC02

Commit message: protoA ERC Pass
Parts:
- removed C10, C8: 100n, symbol Device:C
- removed C9: 2.2u, symbol Device:C
- removed U10: 74LS02, symbol 74xx:74LS02
- removed U2: RaspberryPi_Pico, Module_RaspberryPi_Pico:RaspberryPi_Pico_Common, symbol MCU_Module_RaspberryPi_Pico:RaspberryPi_Pico
- added C14, C7: 100n, symbol Device:C
- added C6: 2.2u, symbol Device:C
- added J1: VIA CE, Connector_PinHeader_1.00mm:PinHeader_1x02_P1.00mm_Vertical, symbol Connector_Generic:Conn_01x02
- added J2: PWR Out, symbol Connector_Generic:Conn_01x04
- added J4: Conn_02x04_Odd_Even, Connector_IDC:IDC-Header_2x04_P2.54mm_Vertical, symbol Connector_Generic:Conn_02x04_Odd_Even
- added R10, R11: 100k, symbol Device:R
- added R8, R9: 22, symbol Device:R
- added U3: RP2040-PICO30, Module_RaspberryPi_Pico:RaspberryPi_Pico_Common, symbol Shared_Library:RP2040-PICO30
- added unit 4 of U4
- added unit 2 of U4
- added unit 3 of U4
- added unit 5 of U4
- added unit 2 of U5
- renumbered C7 to C10, C6 to C11, C5 to C12, C14 to C5, C11 to C8, C12 to C9, R7 to R2, R5 to R3, R6 to R4, R4 to R5, R2 to R6, R3 to R7, U6 to U1, U7 to U10, U1 to U2, U9 to U4, U8 to U5, U5 to U6, U3 to U7, U4 to U8
Connections:
- net +3V3: now also C14.1, C6.1, C7.1, J2.4 (Pin_4), R10.1, R11.1, U3.36 (3V3), U4.14 (VCC)
- net BE0: now also U3.22 (GPIO17)
- net BE1: now also U3.24 (GPIO18)
- net BUS0: now also U3.9 (GPIO6)
- net BUS1: now also U3.10 (GPIO7)
- net BUS2: now also U3.11 (GPIO8)
- net BUS3: now also U3.12 (GPIO9)
- net BUS4: now also U3.14 (GPIO10)
- net BUS5: now also U3.15 (GPIO11)
- net BUS6: now also U3.16 (GPIO12)
- net BUS7: now also U3.17 (GPIO13)
- net CE0: now also R11.2, U3.18 (GPIO25)
- net CE1: now also R10.2, U3.31 (GPIO26_ADC0)
- net CLK: now also R8.2
- net DIR: now also U3.25 (GPIO19)
- net GND: now also C14.2, C6.2, C7.2, J1.2 (Pin_2), J2.1 (Pin_1), J4.7 (Pin_7), U3.3 (GND), U3.38 (GND), U3.8 (GND), U4.7 (GND)
- net PHI2: now also U3.21 (GPIO16)
- net R~{WB}: now also U3.20 (GPIO15)
- net SIO0: now also U3.27 (GPIO21)
- net SIO1: now also U3.29 (GPIO22)
- net SIO2: now also U3.28 (GPIO23)
- net SIO3: now also U3.23 (GPIO24)
- net UART_RX: now also J4.3 (Pin_3), U3.7 (GPIO5)
- net UART_TX: now also J4.5 (Pin_5), U3.6 (GPIO4)
- net ~{IRQB}: now also U3.34 (GPIO28_ADC2)
- net ~{RESB}: now also U3.32 (GPIO27_ADC1)
- net ~{VAB}: now also U3.19 (GPIO14)
- net at U5.7 (O3): now also J1.1 (Pin_1)
- new net: J2.3 (Pin_3), U3.39 (VSYS)
- new net: R9.1, U3.13 (GPIO29)
- new net: R8.1, U3.26 (GPIO20)
- new net +5V: J2.2 (Pin_2), U3.40 (VBUS)
- new net PIX0: J4.2 (Pin_2), U3.1 (GPIO0)
- new net PIX1: J4.4 (Pin_4), U3.2 (GPIO1)
- new net PIX2: J4.6 (Pin_6), U3.4 (GPIO2)
- new net PIX3: J4.8 (Pin_8), U3.5 (GPIO3)
- new net PIXCLK: J4.1 (Pin_1), R9.2
- no-connect marks 1 -> 24
Other:
- note added: "Memory banks"
- note added: "VAB"
- moved on the sheet: C10, C8, C9, U5C

Commit message: protoA PCB done
Parts:
- removed R10, R11: 100k, symbol Device:R
- removed R6, R7: 10k, symbol Device:R
- added C15, C5: 2u2, Capacitor_SMD:C_0603_1608Metric, symbol Device:C
- added FM1, FM2, FM3: Fiducial, Fiducial:Fiducial_1mm_Mask2mm, symbol Mechanical:Fiducial
- added J3: DATA_BUS, Connector_PinHeader_1.00mm:PinHeader_1x08_P1.00mm_Vertical, symbol Connector_Generic:Conn_01x08
- added J4: MEM_DBG, Connector_PinHeader_1.00mm:PinHeader_1x08_P1.00mm_Vertical, symbol Connector_Generic:Conn_01x08
- added J5: CPU_DBG, Connector_PinHeader_1.00mm:PinHeader_1x08_P1.00mm_Vertical, symbol Connector_Generic:Conn_01x08
- added R2: 220R, Resistor_SMD:R_0402_1005Metric, symbol Device:R
- added RN1: 330R, Resistor_SMD:R_Array_Convex_8x0602, symbol Device:R_Pack08
- C1, C12, C3: value 2.2u -> 2u2; footprint (none) -> Capacitor_SMD:C_0603_1608Metric
- C10: renamed from C9; footprint (none) -> Capacitor_SMD:C_0402_1005Metric
- C11, C2, C4: footprint (none) -> Capacitor_SMD:C_0402_1005Metric
- C13: renamed from C14; footprint (none) -> Capacitor_SMD:C_0402_1005Metric
- C14: renamed from C10; footprint (none) -> Capacitor_SMD:C_0402_1005Metric
- C6: renamed from C5; footprint (none) -> Capacitor_SMD:C_0402_1005Metric
- C7: renamed from C6; value 2.2u -> 2u2; footprint (none) -> Capacitor_SMD:C_0603_1608Metric
- C8: renamed from C7; footprint (none) -> Capacitor_SMD:C_0402_1005Metric
- C9: renamed from C8; value 2.2u -> 2u2; footprint (none) -> Capacitor_SMD:C_0603_1608Metric
- J1: renamed from J2; value PWR Out -> PWR_OUT; footprint (none) -> Connector_PinHeader_1.00mm:PinHeader_1x04_P1.00mm_Vertical
- J2: renamed from J1; value VIA CE -> EXT
- J6: renamed from J4; value Conn_02x04_Odd_Even -> PIX
- R1: value 10k -> 220R; footprint (none) -> Resistor_SMD:R_0402_1005Metric
- R3: renamed from R2; value R -> 56k; footprint (none) -> Resistor_SMD:R_0402_1005Metric
- R4: renamed from R3; value R -> 56k; footprint (none) -> Resistor_SMD:R_0402_1005Metric
- R5: renamed from R4; value 3k3 -> 56k; footprint (none) -> Resistor_SMD:R_0402_1005Metric
- R6: renamed from R5; value 3k3 -> 56k; footprint (none) -> Resistor_SMD:R_0402_1005Metric
- R8, R9: value 22 -> 22R; footprint (none) -> Resistor_SMD:R_0402_1005Metric
- U1: renamed from U3; footprint Module_RaspberryPi_Pico:RaspberryPi_Pico_Common -> RaspberryPi_Pico:RaspberryPi_Pico_Common; now not fitted
- U2: footprint Package_DIP:DIP-40_W15.24mm -> Package_DIP:DIP-40_W15.24mm_Socket; Distributor Link (none) -> https://mou.sr/3vFlICu; Manufacturer (none) -> WDC; Manufacturer Part Number (none) -> W65C816S6PG-14
- U3: renamed from U7; Distributor Link (none) -> https://mou.sr/3vCkKqE; Manufacturer (none) -> Adafruit; Manufacturer Part Number (none) -> 4677
- U4: renamed from U8; Distributor Link (none) -> https://mou.sr/3vCkKqE; Manufacturer (none) -> Adafruit; Manufacturer Part Number (none) -> 4677
- U5: renamed from U4; value 74AC02 -> 74LVC02; footprint (none) -> Package_SO:TSSOP-14_4.4x5mm_P0.65mm; Distributor Link (none) -> https://mou.sr/3Udvfdg; Manufacturer (none) -> TI; Manufacturer Part Number (none) -> SN74LVC02APWR
- U6: renamed from U5; value 74HC139 -> 74LVC139; footprint (none) -> Package_SO:TSSOP-16_4.4x5mm_P0.65mm; Distributor Link (none) -> https://mou.sr/3UeJ8aY; Manufacturer (none) -> TI; Manufacturer Part Number (none) -> SN74LVC139APWR
- U7: renamed from U1; value SN74LVC245APW -> 74LVC245; Distributor Link (none) -> https://mou.sr/4alyB3z; Manufacturer (none) -> TI; Manufacturer Part Number (none) -> SN74LVC245APWR
- U8: renamed from U10; value SN74LVC245APW -> 74LVC245; Distributor Link (none) -> https://mou.sr/4alyB3z; Manufacturer (none) -> TI; Manufacturer Part Number (none) -> SN74LVC245APWR
- U9: renamed from U6; value SN74LVC245APW -> 74LVC245; Distributor Link (none) -> https://mou.sr/4alyB3z; Manufacturer (none) -> TI; Manufacturer Part Number (none) -> SN74LVC245APWR
Connections:
- net +3V3: now also C15.1, C5.2; no longer R1.1
- net BE0: now also J5.4 (Pin_4)
- net BE1: now also J5.5 (Pin_5)
- net BUS0: now also RN1.1 (R1.1); no longer U1.9 (GPIO6)
- net BUS1: now also RN1.2 (R2.1); no longer U1.10 (GPIO7)
- net BUS2: now also RN1.3 (R3.1); no longer U1.11 (GPIO8)
- net BUS3: now also RN1.4 (R4.1); no longer U1.12 (GPIO9)
- net BUS4: now also RN1.5 (R5.1); no longer U1.14 (GPIO10)
- net BUS5: now also RN1.6 (R6.1); no longer U1.15 (GPIO11)
- net BUS6: now also RN1.7 (R7.1); no longer U1.16 (GPIO12)
- net BUS7: now also RN1.8 (R8.1); no longer U1.17 (GPIO13)
- net CE0: now also J4.7 (Pin_7)
- net CE1: now also J4.8 (Pin_8)
- net CLK: now also J4.2 (Pin_2)
- net D0: now also J3.1 (Pin_1)
- net D1: now also J3.2 (Pin_2)
- net D2: now also J3.3 (Pin_3)
- net D3: now also J3.4 (Pin_4)
- net D4: now also J3.5 (Pin_5)
- net D5: now also J3.6 (Pin_6)
- net D6: now also J3.7 (Pin_7)
- net D7: now also J3.8 (Pin_8)
- net DIR: now also J5.3 (Pin_3)
- net GND: now also J6.1 (Pin_1), C15.2, C5.1, J4.1 (Pin_1); no longer J2.2 (Pin_2), J6.7 (Pin_7)
- net OE0: no longer R1.2
- net PHI2: now also J5.1 (Pin_1)
- net PIXCLK: now also J6.7 (Pin_7); no longer J6.1 (Pin_1)
- net R~{WB}: now also J5.2 (Pin_2)
- net SIO0: now also J4.3 (Pin_3)
- net SIO1: now also J4.4 (Pin_4)
- net SIO2: now also J4.5 (Pin_5)
- net SIO3: now also J4.6 (Pin_6)
- net UART_RX: now also R2.2; no longer J6.3 (Pin_3)
- net UART_TX: now also R1.2; no longer J6.5 (Pin_5)
- net ~{IRQB}: now also J5.7 (Pin_7)
- net ~{NMIB}: now also J2.2 (Pin_2)
- net ~{RESB}: now also J5.8 (Pin_8)
- net ~{VAB}: now also J5.6 (Pin_6)
- net VSYS: now reaches J1.3 (Pin_3), U1.39 (VSYS)
- net VIA_CE: now reaches J2.1 (Pin_1), U6.7 (O3)
- new net: RN1.10 (R7.2), U1.16 (GPIO12)
- new net: RN1.11 (R6.2), U1.15 (GPIO11)
- new net: RN1.12 (R5.2), U1.14 (GPIO10)
- new net: RN1.13 (R4.2), U1.12 (GPIO9)
- new net: RN1.14 (R3.2), U1.11 (GPIO8)
- new net: RN1.15 (R2.2), U1.10 (GPIO7)
- new net: RN1.16 (R1.2), U1.9 (GPIO6)
- new net: RN1.9 (R8.2), U1.17 (GPIO13)
- new net UART_RX_C: J6.3 (Pin_3), R2.1
- new net UART_TX_C: J6.5 (Pin_5), R1.1
Other:
- note added: "Fiducial markers"
- note added: "Unused"
- moved on the sheet: C13, C14, C7, C9, J2, U5B, U5C, U5D, U5E, U6B, U6C

Commit message: protoA BOM update
Parts:
- C1, C12, C15, C3, C5, C7, C9: Distributor Link (none) -> https://mou.sr/3w2rYEg; Manufacturer (none) -> Samsung; Manufacturer Part Number (none) -> CL10A225KP8NNNC
- C10, C11, C13, C14, C2, C4, C6, C8: Distributor Link (none) -> https://mou.sr/3xGMjjb; Manufacturer (none) -> Samsung; Manufacturer Part Number (none) -> CL05B104KO5VPNC
- J1, J2, J3, J4, J5, U2: now not fitted
- J6: Distributor Link (none) -> https://mou.sr/3Jhh3d6; Manufacturer (none) -> Amphenol FCI; Manufacturer Part Number (none) -> 71600-108LF
- R1, R2: Distributor Link (none) -> https://mou.sr/4aBofNf; Manufacturer (none) -> Panasonic; Manufacturer Part Number (none) -> ERJ-2GEJ221X
- R3, R4, R5, R6: Distributor Link (none) -> https://mou.sr/49zQz12; Manufacturer (none) -> Panasonic; Manufacturer Part Number (none) -> ERJ-2GEJ563X
- R8, R9: Distributor Link (none) -> https://mou.sr/4b0pJA7; Manufacturer (none) -> Panasonic; Manufacturer Part Number (none) -> ERJ-2RKF22R0X

Commit message: Fix J6 PIX connector BOM designator
Parts:
- J6: Distributor Link https://mou.sr/3Jhh3d6 -> https://mou.sr/4b0tdTF; Manufacturer Amphenol FCI -> Molex; Manufacturer Part Number 71600-108LF -> 70246-0801
Changed lines of the file:
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@@
 			)
 		)
-		(property "Distributor Link" "https://mou.sr/3Jhh3d6"
+		(property "Distributor Link" "https://mou.sr/4b0tdTF"
 			(at 173.99 44.45 0)
 			(effects
@@
 			)
 		)
-		(property "Manufacturer Part Number" "71600-108LF"
+		(property "Manufacturer Part Number" "70246-0801"
 			(at 173.99 44.45 0)
 			(effects
@@
 			)
 		)
-		(property "Manufacturer" "Amphenol FCI"
+		(property "Manufacturer" "Molex"
 			(at 173.99 44.45 0)
 			(effects
